Commit message: Changed package name, added display launch file, config file, and added wheels to urdf

File: urdf/robot.urdf (robot description, URDF)
Before this commit: robot jimmy, 5 links, 4 joints
Links:
- added link wheel_center; collision cylinder length=.05 radius=.15; visual cylinder length=.05 radius=.15
- added link wheel_left; collision cylinder length=.05 radius=.2; visual cylinder length=.05 radius=.2
- added link wheel_right; collision cylinder length=.05 radius=.2; visual cylinder length=.05 radius=.2
- link base: geometry collision box size=.94 .78 .198; visual box size=.94 .78 .198
Joints:
- added joint base_wheel_center_joint: type fixed, parent base, child wheel_center, origin xyz=.1 0.0 0.0 rpy=-1.57079 0 0
- added joint base_wheel_left_joint: type fixed, parent base, child wheel_left, origin xyz=-.1 .4 0.0 rpy=-1.57079 0 0
- added joint base_wheel_right_joint: type fixed, parent base, child wheel_right, origin xyz=-.1 -.4 0.0 rpy=-1.57079 0 0

Commit message: Made joints continuous

File: urdf/robot.urdf (robot description, URDF)
Before this commit: robot jimmy, 8 links, 7 joints
Joints:
- joint base_wheel_center_joint: type fixed -> continuous
- joint base_wheel_left_joint: type fixed -> continuous
- joint base_wheel_right_joint: type fixed -> continuous

File: urdf/urdf_from_xacro.urdf (robot description, URDF)
Before this commit: robot jimmy, 8 links, 7 joints
Joints:
- joint base_wheel_center_joint: type fixed -> continuous
- joint base_wheel_left_joint: type fixed -> continuous
- joint base_wheel_right_joint: type fixed -> continuous
