Commit message: Corrected some automatic naming from xacro

File: urdf/robot.xacro (robot description, xacro)
@@ -72,46 +72,4 @@
         </collision>
     </link>
-    <link name="wheel_left">
-        <visual>
-            <origin xyz="-.1 .4 0.0" rpy="-1.57079 0 0" />
-            <geometry>
-                <cylinder radius=".2" length=".05"/>
-            </geometry>
-        </visual>
-        <collision>
-            <origin xyz="-.1 .4 0.0" rpy="-1.57079 0 0" />
-            <geometry>
-                <cylinder radius=".2" length=".05"/>
-            </geometry>
-        </collision>
-    </link>
-    <link name="wheel_right">
-        <visual>
-            <origin xyz="-.1 -.4 0.0" rpy="-1.57079 0 0" />
-            <geometry>
-                <cylinder radius=".2" length=".05"/>
-            </geometry>
-        </visual>
-        <collision>
-            <origin xyz="-.1 -.4 0.0" rpy="-1.57079 0 0" />
-            <geometry>
-                <cylinder radius=".2" length=".05"/>
-            </geometry>
-        </collision>
-    </link>
-    <link name="wheel_center">
-        <visual>
-            <origin xyz=".1 0 0" rpy="-1.57079 0 0" />
-            <geometry>
-                <cylinder radius=".15" length=".05"/>
-            </geometry>
-        </visual>
-        <collision>
-            <origin xyz=".1 0 0" rpy="-1.57079 0 0" />
-            <geometry>
-                <cylinder radius=".15" length=".05"/>
-            </geometry>
-        </collision>
-    </link>
     <joint name="base_laser_vert_bottom_joint" type="fixed">
         <parent link="base"/>
@@ -134,23 +92,8 @@
         <origin xyz=".2325 .0001 1.9201" rpy=".2325 -.0001 1.9201" />
     </joint>
-    <joint name="base_wheel_left_joint" type="fixed">
-        <parent link="base"/>
-        <child link="wheel_left"/>
-        <origin xyz="-.1 .4 0.0" rpy="-1.57079 0 0" />
-    </joint>
-    <joint name="base_wheel_right_joint" type="fixed">
-        <parent link="base"/>
-        <child link="wheel_right"/>
-        <origin xyz="-.1 -.4 0.0" rpy="-1.57079 0 0" />
-    </joint>
-    <joint name="base_wheel_center_joint" type="fixed">
-        <parent link="base"/>
-        <child link="wheel_center"/>
-        <origin xyz=".1 0.0 0.0" rpy="-1.57079 0 0" />
-    </joint>
     <xacro:macro name="wheel_xacro" params="suffix reflect">
-        <link name="wheel_left">
+        <link name="wheel_${suffix}">
             <visual>
-                <origin xyz="-.1 .4 0.0" rpy="-1.57079 0 0" />
+                <origin xyz="-.1 ${reflect * .4} 0.0" rpy="-1.57079 0 0" />
                 <geometry>
                     <cylinder radius=".2" length=".05"/>
@@ -158,5 +101,5 @@
             </visual>
             <collision>
-                <origin xyz="-.1 .4 0.0" rpy="-1.57079 0 0" />
+                <origin xyz="-.1 ${reflect * .4} 0.0" rpy="-1.57079 0 0" />
                 <geometry>
                     <cylinder radius=".2" length=".05"/>
@@ -164,19 +107,13 @@
             </collision>
         </link>
-        <link name="wheel_right">
-            <visual>
-                <origin xyz="-.1 -.4 0.0" rpy="-1.57079 0 0" />
-                <geometry>
-                    <cylinder radius=".2" length=".05"/>
-                </geometry>
-            </visual>
-            <collision>
-                <origin xyz="-.1 -.4 0.0" rpy="-1.57079 0 0" />
-                <geometry>
-                    <cylinder radius=".2" length=".05"/>
-                </geometry>
-            </collision>
-        </link>
-        <link name="wheel_center">
+        <joint name="base_wheel_${suffix}_joint" type="fixed">
+            <parent link="base"/>
+            <child link="wheel_${suffix}"/>
+            <origin xyz="-.1 .4 0.0" rpy="-1.57079 0 0" />
+        </joint>
+    </xacro:macro>
+    <xacro:wheel_xacro suffix="left" reflect="1" />
+    <xacro:wheel_xacro suffix="right" reflect="-1" />
+    <link name="wheel_center">
             <visual>
                 <origin xyz=".1 0 0" rpy="-1.57079 0 0" />
@@ -191,21 +128,9 @@
                 </geometry>
             </collision>
-        </link>
-        <joint name="base_wheel_left_joint" type="fixed">
-            <parent link="base"/>
-            <child link="wheel_left"/>
-            <origin xyz="-.1 .4 0.0" rpy="-1.57079 0 0" />
-        </joint>
-        <joint name="base_wheel_right_joint" type="fixed">
-            <parent link="base"/>
-            <child link="wheel_right"/>
-            <origin xyz="-.1 -.4 0.0" rpy="-1.57079 0 0" />
-        </joint>
-        <joint name="base_wheel_center_joint" type="fixed">
+    </link>
+    <joint name="base_wheel_center_joint" type="fixed">
             <parent link="base"/>
             <child link="wheel_center"/>
             <origin xyz=".1 0.0 0.0" rpy="-1.57079 0 0" />
-        </joint>
-    </xacro:macro>
-    <xacro:wheel_xacro suffix="left" reflect="1" />
+    </joint>
 </robot>

File: urdf/urdf_from_xacro.urdf (robot description, URDF)
Before this commit: robot jimmy, 8 links, 7 joints
Joints:
- joint base_wheel_right_joint: origin xyz=-.1 -.4 0.0 rpy=-1.57079 0 0 -> xyz=-.1 .4 0.0 rpy=-1.57079 0 0

Commit message: adjusted values in urdf file and adjusted launch file to take in GUI argument

File: urdf/robot.xacro (robot description, xacro)
@@ -107,5 +107,5 @@
             </collision>
         </link>
-        <joint name="base_wheel_${suffix}_joint" type="fixed">
+        <joint name="base_wheel_${suffix}_joint" type="continuous">
             <parent link="base"/>
             <child link="wheel_${suffix}"/>
@@ -129,5 +129,5 @@
             </collision>
     </link>
-    <joint name="base_wheel_center_joint" type="fixed">
+    <joint name="base_wheel_center_joint" type="continuous">
             <parent link="base"/>
             <child link="wheel_center"/>

Commit message: Added lidar xacro macros to robot.xacro

File: urdf/robot.xacro (robot description, xacro)
@@ -16,80 +16,12 @@
         </collision>
     </link>
-    <link name="laser_vert_bottom">
-        <visual>
-            <origin xyz=".3158 -.0021 .5100" rpy="3.1355 -1.3045 .0025" />
-            <geometry>
-                <box size =".062 .062 .087"/>
-            </geometry>
-        </visual>
-        <collision>
-            <origin xyz=".3158 -.0021 .5100" rpy="3.1355 -1.3045 .0025" />
-            <geometry>
-                <box size =".062 .062 .087"/>
-            </geometry>
-        </collision>
-    </link>
-    <link name="laser_vert_top_right">
-        <visual>
-            <origin xyz=".2978 -.1450 1.8451" rpy="-1.1760 .6313 -1.9377" />
-            <geometry>
-                <box size =".062 .062 .087"/>
-            </geometry>
-        </visual>
-        <collision>
-            <origin xyz=".2978 -.1450 1.8451" rpy="-1.1760 .6313 -1.9377" />
-            <geometry>
-                <box size =".062 .062 .087"/>
-            </geometry>
-        </collision>
-    </link>
-    <link name="laser_vert_top_left">
-        <visual>
-            <origin xyz=".2997 .1531 1.8443" rpy="1.1780 .6198 1.9560" />
-            <geometry>
-                <box size =".062 .062 .087"/>
-            </geometry>
-        </visual>
-        <collision>
-            <origin xyz=".2997 .1531 1.8443" rpy="1.1780 .6198 1.9560" />
-            <geometry>
-                <box size =".062 .062 .087"/>
-            </geometry>
-        </collision>
-    </link>
-    <link name="laser_horiz">
-        <visual>
-            <origin xyz=".2325 .0001 1.9201" rpy="-.0012068 .114646 -.0015308" />
-            <geometry>
-                <cylinder radius=".052" length=".072"/>
-            </geometry>
-        </visual>
-        <collision>
-            <origin xyz=".2325 .0001 1.9201" rpy="-.0012068 .114646 -.0015308" />
-            <geometry>
-                <cylinder radius=".052" length=".072"/>
-            </geometry>
-        </collision>
-    </link>
-    <joint name="base_laser_vert_bottom_joint" type="fixed">
-        <parent link="base"/>
-        <child link="laser_vert_bottom"/>
-        <origin xyz=".3158 -.0021 .5100" rpy="3.1355 -1.3045 .0025" />
-    </joint>
-    <joint name="base_laser_vert_top_right_joint" type="fixed">
-        <parent link="base"/>
-        <child link="laser_vert_top_right"/>
-          <origin xyz=".2978 -.1450 1.8451" rpy="-1.1760 .6313 -1.9377" />
-    </joint>
-    <joint name="base_laser_vert_top_left_joint" type="fixed">
-        <parent link="base"/>
-        <child link="laser_vert_top_left"/>
-        <origin xyz=".2997 .1531 1.8443" rpy="1.1780 .6198 1.9560" />
-    </joint>
-    <joint name="base_laser_horiz_joint" type="fixed">
-        <parent link="base"/>
-        <child link="laser_horiz"/>
-        <origin xyz=".2325 .0001 1.9201" rpy=".2325 -.0001 1.9201" />
-    </joint>
+    <xacro:include filename="$(find gazebo_plugins)/test/multi_robot_scenario//xacro/laser/hokuyo.xacro" />
+    <xacro:include filename="$(find velodyne_description)/urdf/VLP-16.urdf.xacro"/>
+    <xacro:laser name="laser_vert_bottom" parent="base" xyz="0.3157894464801903 -0.002068548615034871 0.5099999434059285" rpy="3.1354753 -1.3045001 0.0024658" meshes="package://gazebo_plugins/test/multi_robot_scenario/meshes/laser" />
+    <xacro:laser name="laser_vert_top_right" parent="base" xyz=".2978 -.1450 1.8451" rpy="-1.1760 .6313 -1.9377" meshes="package://gazebo_plugins/test/multi_robot_scenario/meshes/laser" />
+    <xacro:laser name="laser_vert_top_left" parent="base" xyz=".2997 .1531 1.8443" rpy="1.1780 .6198 1.9560" meshes="package://gazebo_plugins/test/multi_robot_scenario/meshes/laser" />
+    <VLP-16 parent="base" name="laser_horiz" topic="laser_horiz/packets" hz="10" samples="440" gpu="false">
+        <origin xyz="0.2325416305773505 -0.0001380069427607134 1.920122926231907" rpy="-0.0012068 0.114646 -0.0015308" />
+    </VLP-16>
     <xacro:macro name="wheel_xacro" params="suffix reflect">
         <link name="wheel_${suffix}">

File: urdf/urdf_from_xacro.urdf (robot description, URDF)
Before this commit: robot jimmy, 8 links, 7 joints
Links:
- added link laser_horiz_base_link, mass 0.83; collision cylinder length=0.0717 radius=0.0516; visual mesh filename=package://velodyne_description/meshes/VLP16_base_1.dae
- link laser_horiz: mass None -> 0.01; geometry visual mesh filename=package://velodyne_description/meshes/VLP16_scan.dae
- link laser_vert_bottom: mass None -> 1e-5; geometry collision box size=0.1 0.1 0.1; visual mesh filename=package://gazebo_plugins/test/multi_robot_scenario/meshes/l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
- link laser_vert_top_left: mass None -> 1e-5; geometry collision box size=0.1 0.1 0.1; visual mesh filename=package://gazebo_plugins/test/multi_robot_scenario/meshes/l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
- link laser_vert_top_right: mass None -> 1e-5; geometry collision box size=0.1 0.1 0.1; visual mesh filename=package://gazebo_plugins/test/multi_robot_scenario/meshes/l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
Joints:
- removed joint base_laser_horiz_joint
- added joint laser_horiz_base_mount_joint: type fixed, parent base, child laser_horiz_base_link, origin xyz=0.2325416305773505 -0.0001380069427607134 1.920122926231907 rpy=-0.0012068 0.114646 -0.0015308
- added joint laser_horiz_base_scan_joint: type fixed, parent laser_horiz_base_link, child laser_horiz, origin xyz=0 0 0.0377 rpy=0 0 0
- joint base_laser_vert_bottom_joint: axis (none) -> 0 0 1; origin xyz=.3158 -.0021 .5100 rpy=3.1355 -1.3045 .0025 -> xyz=0.3157894464801903 -0.002068548615034871 0.5099999434059285 rpy=3.1354753 -1.3045001 0.0024658
- joint base_laser_vert_top_left_joint: axis (none) -> 0 0 1
- joint base_laser_vert_top_right_joint: axis (none) -> 0 0 1
